File: hardware/Badge-HackGDL2023.kicad_sch (KiCad schematic)
At the start: 14 parts, among them J1 SWD, SW1 SW_RST, SW2 On, U1 PY32F002AA15M6TU

Commit message: Update BOM
Parts:
- BT1: LCSC# (none) -> C964833; manf# BAT-HLD-001 -> (none)
Changed lines of the file:
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@@
       (effects (font (size 1.27 1.27)))
     )
-    (property "LCSC#" "" (at 123.19 50.8 0)
+    (property "LCSC#" "C964833" (at 123.19 50.8 0)
       (effects (font (size 1.27 1.27)) hide)
     )
-    (property "manf#" "BAT-HLD-001" (at 123.19 50.8 0)
+    (property "manf#" "" (at 123.19 50.8 0)
       (effects (font (size 1.27 1.27)) hide)
     )

Commit message: update v1.0
Connections:
- net SWCLK: now also J1.3 (Pin_3); no longer J1.2 (Pin_2)
- net SWDIO: now also J1.2 (Pin_2); no longer J1.3 (Pin_3)
Changed lines of the file:
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@@
     (effects (font (size 1.27 1.27)) (justify left bottom))
   )
-  (label "SWDIO" (at 62.611 88.9 0) (fields_autoplaced)
+  (label "SWDIO" (at 62.611 86.36 0) (fields_autoplaced)
     (effects (font (size 1.27 1.27)) (justify left bottom))
   )
@@
     (effects (font (size 1.27 1.27)) (justify left bottom))
   )
-  (label "SWCLK" (at 62.611 86.36 0) (fields_autoplaced)
+  (label "SWCLK" (at 62.611 88.9 0) (fields_autoplaced)
     (effects (font (size 1.27 1.27)) (justify left bottom))
   )
